File: LowNoise5V - HW Files/LowNoise5V.sch (KiCad schematic (older format))
At the start: 12 parts, among them J1 USB_A, J2 Conn_01x02

Commit message: Finalize Routing
Parts:
- Acc1: footprint LowNoise5V:FuseHolder -> (none)
- F1: footprint (none) -> LowNoise5V:FuseHolder
- J2: footprint TerminalBlock:TerminalBlock_bornier-2_P5.08mm -> LowNoise5V:1935161
Changed lines of the file:
@@
 	1    0    0    -1
 $EndComp
-Wire Wire Line
-	6400 1500 7050 1500
-Wire Wire Line
-	7050 1700 6400 1700
 $Comp
 L Device:C C1
@@
 F 0 "F1" V 2303 1000 50  0000 C CNN
 F 1 "500mA 250VAC Fast Blow" V 2394 1000 50  0000 C CNN
-F 2 "" V 2430 1000 50  0001 C CNN
+F 2 "LowNoise5V:FuseHolder" V 2430 1000 50  0001 C CNN
 F 3 "~" H 2500 1000 50  0001 C CNN
 F 4 "Xucheng Elec" H 2500 1000 50  0001 C CNN "Part 1 MF"
@@
 F 0 "Acc1" H 2641 1421 50  0000 L CNN
 F 1 "Fuse Holder" H 2641 1330 50  0000 L CNN
-F 2 "LowNoise5V:FuseHolder" H 2512 1300 50  0001 C CNN
+F 2 "" H 2512 1300 50  0001 C CNN
 F 3 "~" H 2512 1300 50  0001 C CNN
 F 4 "HONGJU" H 2500 1300 50  0001 C CNN "Part 1 MF"
@@
 	1200 2800 1200 2900
 Connection ~ 1200 2900
-Wire Wire Line
-	5150 1500 6000 1500
-Wire Wire Line
-	5150 1700 6000 1700
 $Comp
 L Device:CP C3
@@
 F 0 "J2" H 1218 1767 50  0000 C CNN
 F 1 "Conn_01x02" H 1218 1676 50  0000 C CNN
-F 2 "TerminalBlock:TerminalBlock_bornier-2_P5.08mm" H 1300 1550 50  0001 C CNN
+F 2 "LowNoise5V:1935161" H 1300 1550 50  0001 C CNN
 F 3 "~" H 1300 1550 50  0001 C CNN
 	1    1300 1550
@@
 Wire Wire Line
 	1850 2200 3200 2200
+Wire Wire Line
+	5150 1500 6000 1500
+Wire Wire Line
+	6400 1500 7050 1500
+Wire Wire Line
+	5150 1700 6000 1700
+Wire Wire Line
+	6400 1700 7050 1700
 $EndSCHEMATC
