File: LowNoise5V - HW Files/LowNoise5V.kicad_pcb (KiCad board)
At the start: 2 copper layers, 81 x 54 mm, 15 parts, among them J1 USB_A, J2 Conn_01x02

Commit message: Finalize Artwork
Parts:
- added G***: LOGO, LowNoise5V:artwork_top, F.Cu at (40.5, 27.0)
- added G***: LOGO, LowNoise5V:artwork_bottom, B.Cu at (40.5, 27.0)
Routing:
- net (no net): track 0.00 -> 3.41 mm
