File: LowNoise5V - HW Files/LowNoise5V.kicad_pcb (KiCad board)
At the start: 2 copper layers, 81 x 54 mm, 17 parts, among them J1 USB_A, J2 Conn_01x02

Commit message: Finalize design files for release
Other:
- board text added: "JLCJLCJLCJLC"
- board text added: "Order Number"
